File: layout/source/source_bt_rev_a.brd (EAGLE design)
At the start: 24 x 45 mm, 22 parts, among them IC1 LP2985-SOT23-5, IC2 IC_USBLC6-2, IC3 HM-10

Commit message: Changed structure, added HM-11
Parts:
- C1, C2, C3: value 100n -> 1µF
- R6: value 1k -> 10k
Changed lines of the file:
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@@
 </element>
 <element name="TRS1" library="con-trs" package="YD-PJ-3504" value="PJ-3504" x="7" y="0" rot="R90"/>
-<element name="C3" library="rcl" package="C0603" value="100n" x="7.5" y="15" smashed="yes">
+<element name="C3" library="rcl" package="C0603" value="1µF" x="7.5" y="15" smashed="yes">
 <attribute name="NAME" x="9.115" y="14.635" size="0.8128" layer="25"/>
 </element>
@@
 <attribute name="VALUE" x="14.542" y="11.65" size="0.4064" layer="27" ratio="10" rot="R90"/>
 </element>
-<element name="C1" library="rcl" package="C0603" value="100n" x="13.75" y="10" smashed="yes" rot="R180">
+<element name="C1" library="rcl" package="C0603" value="1µF" x="13.75" y="10" smashed="yes" rot="R180">
 <attribute name="NAME" x="12.135" y="10.365" size="0.8128" layer="25" rot="R180"/>
 </element>
-<element name="C2" library="rcl" package="C0603" value="100n" x="11" y="13.5" smashed="yes" rot="R270">
+<element name="C2" library="rcl" package="C0603" value="1µF" x="11" y="13.5" smashed="yes" rot="R270">
 <attribute name="NAME" x="11.365" y="15.115" size="0.8128" layer="25" rot="R90"/>
 </element>
-<element name="R6" library="rcl" package="R0603" value="1k" x="21" y="24" smashed="yes">
+<element name="R6" library="rcl" package="R0603" value="10k" x="21" y="24" smashed="yes">
 <attribute name="NAME" x="20.365" y="22.385" size="0.8128" layer="25"/>
 </element>
