File: layout/display/d150_in14.brd (EAGLE design)
At the start: 100 x 42 mm, 69 parts, among them IC1 STM32F103C8T, IC2 LP2985-SOT23-5, IC3 IC_USBLC6-2, IC4 IC_USBLC6-2, IC5 LT1619ES8, IC6 LP2985-SOT23-5, IC7 IRF7470, T1 LPISR, Y1 532-CRYSTAL, Y2 EQ161-CRYSTAL

Commit message: Changed structure, added c150 and c200
Parts:
- removed BAT1: (no value), battery-holder:HARWIN-CR1220
- removed BT: HM-11, bt:HM-11
- removed C10, C11: 10µF/6.3V, rcl:C0603
- removed C12: 22nF, rcl:C0603
- removed C13, C14: 10p, rcl:C0603
- removed C15, C16, C22: 10µF, rcl:C0603
- removed C17: 100µF/6.3V, rcl:C1210
- removed C18, C19, C20, C21: 100nF, rcl:C0603
- removed C9: 150pF, rcl:C0603
- removed D2: BAT54C, diode:SOT23
- removed D3: ES2, diode:DO-214AA
- removed F1, R12, R13, R7: 1k, rcl:R0603
- removed FB1: EMI, rcl:R0603
- removed ISP: TACT-SWITCH-40-40, tactile-switch:40-40
- removed LED1, LED2, LED3: (no value), led:CHIP-LED0603
- removed LOGO1: OSHW_LOGO_FILLX0200-NT, ohw-logo:OSHW_FILLX200_NOTEXT
- removed R18: 82k, rcl:R0603
- removed R19: 1M, rcl:M1206
- removed R23: 0.01R, rcl:R1206
- removed R5: 33R, rcl:R0603
- removed R6: 1k5, rcl:R0603
- removed R8: 10k, rcl:R0603
- removed SWD: (no value), microbuilder:1X05_ROUND
- removed TP1, TP2, TP3, TP4: (no value), microbuilder:TESTPOINT_ROUND_2MM
- removed TRS1: PJ-3504, con-trs:YD-PJ-3504
- removed X1: (no value), con-cypressindustries:32005-201
- removed Y1: 532-CRYSTAL, euroquartz:2PIN50X32
- removed Y2: EQ161-CRYSTAL, euroquartz:EQ161
- added GL1, GL2, GL3, GL4: (no value), nixie_tube:NE2-NEON-BULB-DRILL
- added IC8: 74HC595D, 74xx-eu:SO16
- added JP2: (no value), con-pinhead:2X03SMD
- added N1, U$7, U$8, U$9: IN-14, nixietubes-russian:IN-14
- added R10, R30, R40, R50, R60: (no value), rcl:R0603
- added RN10, RN11, RN20, RN21, RN30, RN31, RN40, RN41, RN50, RN51, RN60, RN61, RN70, RN71, RN80, RN81: (no value), resistor-net:CTS742C083
- added T10, T11, T12, T13, T14, T15, T16, T17, T18, T19, T2, T20, T21, T22, T23, T24, T25, T26, T27, T28, T29, T3, T30, T31, T32, T33, T34, T35, T36, T37, T38, T39, T4, T40, T41, T42, T43, T44, T45, T46, T47, T48, T49, T50, T51, T52, T53, T54, T55, T56, T57, T58, T59, T60, T61, T62, T63, T64, T65, T66, T67, T68, T69: (no value), transistor-hv:SOT23
- added U$3: (no value), pcb-artwork:GITHUB/JAN1S
- C1, C2: value 10p -> (none)
- C3, C5, C6: value 10µF/6.3V -> (none)
- C4: value 1µF/250V -> (none); device rcl:C2220K -> rcl:C0603
- C7, C8: value 10nF -> (none)
- IC1: value STM32F103C8T -> 74HC595D; device micro-stm_v3:LQFP48 -> 74xx-eu:SO16
- IC2, IC6: value LP2985-SOT23-5 -> 74HC595D; device vreg:SOT23-5 -> 74xx-eu:SO16
- IC3, IC4: value IC_USBLC6-2 -> 74HC595D; device dp_devices:SOT-23-6L -> 74xx-eu:SO16
- IC5: value LT1619ES8 -> 74HC595D; device lt:SO8 -> 74xx-eu:SO16
- IC7: value IRF7470 -> 74HC595D; device ir:SO8 -> 74xx-eu:SO16
- JP1: device con-pinhead:2X05SMD -> con-pinhead:2X03SMD
- R1, R2, R3, R4: value 33R -> (none)
- R20: value 8k2 -> (none)
- T1: value LPISR -> (none); device fastron:PISR -> transistor-hv:SOT23
- U$1: device pcb-artwork:JANIS_10MM -> ohw-logo:OSHW_FILLX200_NOTEXT
- U$5, U$6: value (none) -> IN-14; device pcb-artwork:GITHUB/JAN1S -> nixietubes-russian:IN-14
- moved U$5 102.0 mm to (113.0, 26.5)
- moved T1 86.4 mm to (101.0, 31.5), turned to 180 degrees
- moved R20 76.1 mm to (113.0, 18.3), turned to 270 degrees
- moved C1 69.8 mm to (140.0, 5.00), turned to 90 degrees
- moved C2 56.2 mm to (127.5, 5.00), turned to 90 degrees
- moved IC1 55.5 mm to (134.0, 7.50)
- moved C4 54.6 mm to (91.0, 5.00), turned to 90 degrees
- moved C8 54.3 mm to (21.0, 5.00)
- moved IC5 50.1 mm to (65.0, 7.50)
- moved C7 47.7 mm to (33.5, 5.00), turned to 90 degrees
- moved IC2 42.8 mm to (121.5, 7.50), turned to 180 degrees
- moved C3 40.8 mm to (115.2, 4.99)
- moved U$1 37.5 mm to (73.0, 4.00)
- moved U$2 37.5 mm to (92.0, 8.00), flipped to the top
- moved U$6 37.5 mm to (85.0, 26.5), flipped to the top
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Connections:
- removed net +3V3: BT.9, C18.1, C19.1, C20.1, C21.1, C22.1, C6.1, IC1.24, IC1.36, IC1.48, IC1.9, IC2.5, IC3.5, LED1.A, LED2.A, R5.2, R6.1, R8.1
- removed net ASDAWJIODJA: R5.1, SWD.4
- removed net BT_USER: BT.16, IC1.11, R8.2
- removed net HV_EN: IC1.18, IC5.1
- removed net HV_VCC: C4.1, D3.C, JP1.2, R19.2
- removed net I2C1_SCL: IC1.42
- removed net I2C1_SDA: IC1.43
- removed net I2C2_SCL: IC1.21
- removed net I2C2_SDA: IC1.22
- removed net JNTRST: IC1.40
- removed net JTDI: IC1.38
- removed net JTDO: IC1.39
- removed net LED_BOOT: IC1.46, R13.1
- removed net LED_FIX: IC1.45, R12.1
- removed net N$22: F1.2, FB1.2
- removed net N$23: IC3.1, R2.2
- removed net N$24: R2.1, X1.2
- removed net N$25: IC4.4, R4.2
- removed net N$26: BT.15, R7.1
- removed net N$27: LED3.A, R7.2
- removed net N$28: R3.1, TRS1.5
- removed net N$29: C13.1, IC1.4, Y2.P$1
- removed net N$30: C14.1, IC1.3, Y2.P$2
- removed net N$32: IC1.19
- removed net N$34: IC1.20
- removed net N$36: R1.1, X1.3
- removed net N$38: IC1.29
- removed net N$42: IC1.10
- removed net N$48: IC1.41
- removed net N$55: IC1.25
- removed net NX_EN: IC1.14, JP1.8
- removed net NX_RCK: IC1.16, JP1.10
- removed net RESET: IC1.7, ISP.3, ISP.4, SWD.5
- removed net RTC-TAMPER: IC1.2
- removed net SPI1_MOSI: IC1.17, JP1.7
- removed net SPI1_SCK: IC1.15, JP1.9
- removed net SPI2_MISO: IC1.27
- removed net SPI2_MOSI: IC1.28
- removed net SPI2_SCK: IC1.26
- removed net SWCLK: IC1.37, SWD.2
- removed net SWDIO: IC1.34, SWD.3
- removed net TRS_VCC: C10.1, IC4.5, IC6.5, TRS1.4
- removed net USART1_RX: IC1.31, IC4.1
- removed net USART1_TX: IC1.30, IC4.3
- removed net USART2_RX: BT.2, IC1.13
- removed net USART2_TX: BT.4, IC1.12
- removed net USB_DM: IC1.32, IC3.6
- removed net USB_DP: IC1.33, IC3.4
- removed net VBAT: BAT1.POS, C11.1, IC1.1
- new net 1A: IC1.15, RN10.4
- new net 1B: IC1.1, RN10.3
- new net 1C: IC1.2, RN10.2
- new net 1D: IC1.3, RN10.1
- new net 1E: IC1.4, RN11.4
- new net 1F: IC1.5, RN11.3
- new net 1G: IC1.6, RN11.2
- new net 1H: IC1.7, RN11.1
- new net 2A: IC2.15, RN20.4
- new net 2B: IC2.1, RN20.3
- new net 2B0: RN30.7, T20.1
- new net 2B1: RN30.8, T21.1
- new net 2B2: RN20.7, T22.1
- new net 2B3: RN20.8, T23.1
- new net 2B4: RN21.5, T24.1
- new net 2B5: RN21.6, T25.1
- new net 2B6: RN21.7, T26.1
- new net 2B7: RN21.8, T27.1
- new net 2B8: RN30.5, T28.1
- new net 2B9: RN30.6, T29.1
- new net 2C: IC2.2, RN20.2
- new net 2D: IC2.3, RN20.1
- new net 2E: IC2.4, RN21.4
- new net 2F: IC2.5, RN21.3
- new net 2G: IC2.6, RN21.2
- new net 2H: IC2.7, RN21.1
- new net 3A: IC3.15, RN30.4
- new net 3B: IC3.1, RN30.3
- new net 3B0: RN41.7, T30.1
- new net 3B1: RN41.8, T31.1
- new net 3B2: RN31.7, T32.1
- new net 3B3: RN31.8, T33.1
- new net 3B4: RN40.5, T34.1
- new net 3B5: RN40.6, T35.1
- new net 3B6: RN40.7, T36.1
- new net 3B7: RN40.8, T37.1
- new net 3B8: RN41.5, T38.1
- new net 3B9: RN41.6, T39.1
- new net 3C: IC3.2, RN30.2
- new net 3D: IC3.3, RN30.1
- new net 3E: IC3.4, RN31.4
- new net 3F: IC3.5, RN31.3
- new net 3G: IC3.6, RN31.2
- new net 3H: IC3.7, RN31.1
- new net 4A: IC4.15, RN40.4
- new net 4B: IC4.1, RN40.3
- new net 4B0: RN60.5, T40.1
- new net 4B1: RN60.6, T41.1
- new net 4B2: RN50.5, T42.1
- new net 4B3: RN50.6, T43.1
- new net 4B4: RN50.7, T44.1
- new net 4B5: RN50.8, T45.1
- new net 4B6: RN51.5, T46.1
- new net 4B7: RN51.6, T47.1
- new net 4B8: RN51.7, T48.1
- new net 4B9: RN51.8, T49.1
- new net 4C: IC4.2, RN40.2
- new net 4D: IC4.3, RN40.1
- new net 4E: IC4.4, RN41.4
- new net 4F: IC4.5, RN41.3
- new net 4G: IC4.6, RN41.2
- new net 4H: IC4.7, RN41.1
- new net 5A: IC5.15, RN50.4
- new net 5B: IC5.1, RN50.3
- new net 5B0: RN71.5, T50.1
- new net 5B1: RN71.6, T51.1
- new net 5B2: RN61.5, T52.1
- new net 5B3: RN61.6, T53.1
- new net 5B4: RN61.7, T54.1
- new net 5B5: RN61.8, T55.1
- new net 5B6: RN70.5, T56.1
- new net 5B7: RN70.6, T57.1
- new net 5B8: RN70.7, T58.1
- new net 5B9: RN70.8, T59.1
- new net 5C: IC5.2, RN50.2
- new net 5D: IC5.3, RN50.1
- new net 5E: IC5.4, RN51.4
- new net 5F: IC5.5, RN51.3
- new net 5G: IC5.6, RN51.2
- new net 5H: IC5.7, RN51.1
- new net 6A: IC6.15, RN60.4
- new net 6B: IC6.1, RN60.3
- new net 6B0: RN81.7, T60.1
- new net 6B1: RN81.8, T61.1
- new net 6B2: RN71.7, T62.1
- new net 6B3: RN71.8, T63.1
- new net 6B4: RN80.5, T64.1
- new net 6B5: RN80.6, T65.1
- new net 6B6: RN80.7, T66.1
- new net 6B7: RN80.8, T67.1
- new net 6B8: RN81.5, T68.1
- new net 6B9: RN81.6, T69.1
- new net 6C: IC6.2, RN60.2
- new net 6D: IC6.3, RN60.1
- new net 6E: IC6.4, RN61.4
- new net 6F: IC6.5, RN61.3
- new net 6G: IC6.6, RN61.2
- new net 6H: IC6.7, RN61.1
- new net 7A: IC7.15, RN70.4
- new net 7B: IC7.1, RN70.3
- new net 7C: IC7.2, RN70.2
- new net 7D: IC7.3, RN70.1
- new net 7E: IC7.4, RN71.4
- new net 7F: IC7.5, RN71.3
- new net 7G: IC7.6, RN71.2
- new net 7H: IC7.7, RN71.1
- new net 8A: IC8.15, RN80.4
- new net 8B: IC8.1, RN80.3
- new net 8C: IC8.2, RN80.2
- new net 8D: IC8.3, RN80.1
- new net 8E: IC8.4, RN81.4
- new net 8F: IC8.5, RN81.3
- new net 8G: IC8.6, RN81.2
- new net 8H: IC8.7, RN81.1
- new net EN: IC1.13, IC2.13, IC3.13, IC4.13, IC5.13, IC6.13, IC7.13, IC8.13, JP1.1
- new net GL1: RN31.5, T1.1
- new net GL2: RN31.6, T2.1
- new net GL3: RN60.7, T3.1
- new net GL4: RN60.8, T4.1
- new net MOSI: IC1.14, JP1.4
- new net N$21: GL1.1, R1.1
- new net N$6: GL1.2, T1.3
- new net N1_B0: RN20.6, T11.1
- new net N1_B1: RN10.5, T12.1
- new net N1_B2: RN10.6, T13.1
- new net N1_B3: RN10.7, T14.1
- new net N1_B4: RN10.8, T15.1
- new net N1_B5: RN11.5, T16.1
- new net N1_B6: RN11.6, T17.1
- new net N1_B7: RN11.7, T18.1
- new net N1_B8: RN11.8, T19.1
- new net N1_B9: RN20.5, T10.1
- new net N1_DP: N1.2
- new net N1_IC: N1.13
- new net N1_K0: N1.12, T11.3
- new net N1_K1: N1.3, T12.3
- new net N1_K2: N1.4, T13.3
- new net N1_K3: N1.5, T14.3
- new net N1_K4: N1.6, T15.3
- new net N1_K5: N1.7, T16.3
- new net N1_K6: N1.8, T17.3
- new net N1_K7: N1.9, T18.3
- new net N1_K8: N1.10, T19.3
- new net N1_K9: N1.11, T10.3
- new net N2_0: T22.3, U$5.3
- new net N2_1: T21.3, U$5.12
- new net N2_2: T20.3, U$5.11
- new net N2_3: T29.3, U$5.10
- new net N2_4: T28.3, U$5.9
- new net N2_5: T27.3, U$5.8
- new net N2_6: T26.3, U$5.7
- new net N2_7: T25.3, U$5.6
- new net N2_8: T24.3, U$5.5
- new net N2_9: T23.3, U$5.4
- new net N3_0: T32.3, U$6.3
- new net N3_1: T31.3, U$6.12
- new net N3_2: T30.3, U$6.11
- new net N3_3: T39.3, U$6.10
- new net N3_4: T38.3, U$6.9
- new net N3_5: T37.3, U$6.8
- new net N3_6: T36.3, U$6.7
- new net N3_7: T35.3, U$6.6
- new net N3_8: T34.3, U$6.5
- new net N3_9: T33.3, U$6.4
- new net N4_0: T42.3, U$7.3
- new net N4_1: T41.3, U$7.12
- new net N4_2: T40.3, U$7.11
- new net N4_3: T49.3, U$7.10
- new net N4_4: T48.3, U$7.9
- new net N4_5: T47.3, U$7.8
- new net N4_6: T46.3, U$7.7
- new net N4_7: T45.3, U$7.6
- new net N4_8: T44.3, U$7.5
- new net N4_9: T43.3, U$7.4
- new net N5_0: T52.3, U$8.3
- new net N5_1: T51.3, U$8.12
- new net N5_2: T50.3, U$8.11
- new net N5_3: T59.3, U$8.10
- new net N5_4: T58.3, U$8.9
- new net N5_5: T57.3, U$8.8
- new net N5_6: T56.3, U$8.7
- new net N5_7: T55.3, U$8.6
- new net N5_8: T54.3, U$8.5
- new net N5_9: T53.3, U$8.4
- new net N6_0: T62.3, U$9.3
- new net N6_1: T61.3, U$9.12
- new net N6_2: T60.3, U$9.11
- new net N6_3: T69.3, U$9.10
- new net N6_4: T68.3, U$9.9
- new net N6_5: T67.3, U$9.8
- new net N6_6: T66.3, U$9.7
- new net N6_7: T65.3, U$9.6
- new net N6_8: T64.3, U$9.5
- new net N6_9: T63.3, U$9.4
- new net RCK: IC1.12, IC2.12, IC3.12, IC4.12, IC5.12, IC6.12, IC7.12, IC8.12, JP1.5
- new net SCK: IC1.11, IC2.11, IC3.11, IC4.11, IC5.11, IC6.11, IC7.11, IC8.11, JP1.3
- new net SCL: IC1.10, IC2.10, IC3.10, IC4.10, IC5.10, IC6.10, IC7.10, IC8.10, JP1.2
- new net VDD: JP2.1, R1.2, R10.2, R2.2, R20.2, R3.2, R30.2, R4.2, R40.2, R50.2, R60.2
- net +5V: now also C1.1, C2.1, C4.1, C6.1, C7.1, C8.1, IC1.16, IC2.16, IC3.16, IC4.16, IC5.16, IC6.16, IC7.16, IC8.16, JP2.6; no longer C15.1, C17.1, D2.2, FB1.1, IC2.1, IC2.3, IC5.8, IC6.1, IC6.3, JP1.5, TP1.P$1
- net GND: now also IC2.8, IC3.8, IC4.8, IC5.8, IC6.8, IC7.8, IC8.8, JP2.2, JP2.3, JP2.4, JP2.5, T1.2, T10.2, T11.2, T12.2, T13.2, T14.2, T15.2, T16.2, T17.2, T18.2, T19.2, T2.2, T20.2, T21.2, T22.2, T23.2, T24.2, T25.2, T26.2, T27.2, T28.2, T29.2, T3.2, T30.2, T31.2, T32.2, T33.2, T34.2, T35.2, T36.2, T37.2, T38.2, T39.2, T4.2, T40.2, T41.2, T42.2, T43.2, T44.2, T45.2, T46.2, T47.2, T48.2, T49.2, T50.2, T51.2, T52.2, T53.2, T54.2, T55.2, T56.2, T57.2, T58.2, T59.2, T60.2, T61.2, T62.2, T63.2, T64.2, T65.2, T66.2, T67.2, T68.2, T69.2; no longer BAT1.NEG, BT.12, C10.2, C11.2, C12.2, C13.2, C14.2, C15.2, C16.2, C17.2, C18.2, C19.2, C20.2, C21.2, C22.2, C9.2, IC1.23, IC1.35, IC1.44, IC1.47, IC2.2, IC3.2, IC4.2, IC5.4, IC6.2, ISP.1, ISP.2, JP1.1, JP1.3, JP1.4, LED3.C, R20.2, R23.1, SWD.1, T1.P$2, TP4.P$1, TRS1.3, X1.5, X1.M1, X1.M2, X1.M3, X1.M4
- net N$1: now also GL2.1, R2.1; no longer C1.1, IC1.6, Y1.P$1
- net N$10: now also IC1.9, IC2.14; no longer LED2.C, R13.2
- net N$11: now also IC2.9, IC3.14; no longer LED1.C, R12.2
- net N$12: now also IC3.9, IC4.14; no longer R4.1, TRS1.2
- net N$13: now also R30.1, U$6.1; no longer IC7.5, IC7.6, IC7.7, IC7.8, TP2.P$1
- net N$14: now also R40.1, U$7.1; no longer C12.1, IC5.3, R18.1
- net N$15: now also R60.1, U$9.1; no longer C9.1, R18.2
- net N$16: now also IC4.9, IC5.14; no longer D3.A, T1.P$1
- net N$17: now also R50.1, U$8.1; no longer IC5.2, R19.1, R20.1
- net N$18: now also IC5.9, IC6.14; no longer IC5.5, IC7.1, IC7.2, IC7.3, R23.2
- net N$19: now also IC6.9, IC7.14; no longer C16.1, D2.3, IC5.7
- net N$2: now also GL3.1, R3.1; no longer C2.1, IC1.5, Y1.P$2
- net N$20: now also IC7.9, IC8.14; no longer C7.1, IC2.4
- net N$3: now also GL4.1, R4.1; no longer F1.1, X1.1
- net N$4: now also N1.1, R10.1; no longer C8.1, IC6.4
- net N$5: now also GL2.2, T2.3; no longer IC3.3, R1.2, R6.2
- net N$7: now also GL4.2, T4.3; no longer IC4.6, R3.2
- net N$8: now also GL3.2, T3.3; no longer D2.1, TP3.P$1
- net N$9: now also R20.1, U$5.1; no longer IC5.6, IC7.4
Routing:
- net EN: track 0.00 -> 161.6 mm, vias 0 -> 9
- net RCK: track 0.00 -> 154.3 mm, vias 0 -> 9
- net SCK: track 0.00 -> 153.1 mm, vias 0 -> 9
- net SCL: track 0.00 -> 148.9 mm, vias 0 -> 9
- net VDD: track 0.00 -> 143.1 mm
- net +3V3: track 103.3 -> 0.00 mm, vias 4 -> 0
- net MOSI: track 0.00 -> 93.4 mm, vias 0 -> 2
- net HV_EN: track 76.1 -> 0.00 mm, vias 2 -> 0
- net GND: track 0.00 -> 53.7 mm, vias 316 -> 198
- net USART2_TX: track 48.3 -> 0.00 mm, vias 4 -> 0
- net USART2_RX: track 47.7 -> 0.00 mm, vias 2 -> 0
- net SPI1_MOSI: track 42.4 -> 0.00 mm
- net RESET: track 39.3 -> 0.00 mm, vias 2 -> 0
- net BT_USER: track 38.1 -> 0.00 mm
- net SPI1_SCK: track 37.5 -> 0.00 mm
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- removed copper zone on layer 1, net +5V
Other:
- board size 100 x 42 mm -> 150 x 42 mm
- board text removed: "GND"
- board text removed: "RST"
- board text removed: "SWCLK"
- board text removed: "SWDIO"
- board text removed: "VCC"
