File: layout/display/d100_zm1000_rev_b.brd (EAGLE design)
At the start: 100 x 42 mm, 86 parts, among them IC1 74HC595PW, IC2 74HC595PW, IC3 74HC595PW, IC4 74HC595PW, IC5 74HC595PW, IC6 74HC595PW

Commit message: Fixed naming
Connections:
- net 4C0 renamed N4_0
- net 4C1 renamed N4_1
- net 4C2 renamed N4_2
- net 4C3 renamed N4_3
- net 4C4 renamed N4_4
- net 4C5 renamed N4_5
- net 4C6 renamed N4_6
- net 4C7 renamed N4_7
- net 4C8 renamed N4_8
- net 4C9 renamed N4_9
Changed lines of the file:
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@@
 <wire x1="16" y1="16" x2="17.75" y2="14.25" width="0.254" layer="16"/>
 </signal>
-<signal name="4C0">
+<signal name="N4_0">
 <contactref element="T40" pad="3"/>
 <contactref element="N4" pad="K0"/>
@@
 <wire x1="11.2" y1="30" x2="9.1" y2="30" width="0.254" layer="1"/>
 </signal>
-<signal name="4C1">
+<signal name="N4_1">
 <contactref element="T41" pad="3"/>
 <contactref element="N4" pad="K1"/>
@@
 <wire x1="16.27" y1="32.67" x2="17" y2="33.4" width="0.254" layer="1"/>
 </signal>
-<signal name="4C2">
+<signal name="N4_2">
 <contactref element="T42" pad="3"/>
 <contactref element="N4" pad="K2"/>
@@
 <wire x1="20.5" y1="33.5" x2="20.5" y2="33.4" width="0.254" layer="1"/>
 </signal>
-<signal name="4C3">
+<signal name="N4_3">
 <contactref element="T43" pad="3"/>
 <contactref element="N4" pad="K3"/>
@@
 <wire x1="18.8" y1="30" x2="20.9" y2="30" width="0.254" layer="1"/>
 </signal>
-<signal name="4C4">
+<signal name="N4_4">
 <contactref element="T44" pad="3"/>
 <contactref element="N4" pad="K4"/>
@@
 <wire x1="20.8" y1="26.6" x2="20.9" y2="26.5" width="0.254" layer="1"/>
 </signal>
-<signal name="4C5">
+<signal name="N4_5">
 <contactref element="T45" pad="3"/>
 <contactref element="N4" pad="K5"/>
@@
 <wire x1="20.2" y1="20.7" x2="20.9" y2="20" width="0.254" layer="1"/>
 </signal>
-<signal name="4C6">
+<signal name="N4_6">
 <contactref element="T46" pad="3"/>
 <contactref element="N4" pad="K6"/>
@@
 <wire x1="9.7" y1="20.6" x2="9.1" y2="20" width="0.254" layer="1"/>
 </signal>
-<signal name="4C7">
+<signal name="N4_7">
 <contactref element="T47" pad="3"/>
 <contactref element="N4" pad="K7"/>
@@
 <wire x1="9.1" y1="26.2" x2="9.1" y2="25.5" width="0.254" layer="1"/>
 </signal>
-<signal name="4C8">
+<signal name="N4_8">
 <contactref element="T48" pad="3"/>
 <contactref element="N4" pad="K8"/>
@@
 <wire x1="13.73" y1="32.67" x2="13" y2="33.4" width="0.254" layer="1"/>
 </signal>
-<signal name="4C9">
+<signal name="N4_9">
 <contactref element="T49" pad="3"/>
 <contactref element="N4" pad="K9"/>
