File: layout/display/d100_zm1000_rev_b.sch (EAGLE design)
At the start: 83 parts, among them IC1 74HC595PW, IC2 74HC595PW, IC3 74HC595PW, IC4 74HC595PW, IC5 74HC595PW, IC6 74HC595PW, T1 SMBTA42, T10 SMBTA42, T11 SMBTA42, T12 SMBTA42, T13 SMBTA42, T14 SMBTA42, T15 SMBTA42, T16 SMBTA42, T17 SMBTA42, T18 SMBTA42, T19 SMBTA42, T2 SMBTA42, T20 SMBTA42, T21 SMBTA42, T22 SMBTA42, T23 SMBTA42, T24 SMBTA42, T25 SMBTA42, T26 SMBTA42, T27 SMBTA42, T28 SMBTA42, T29 SMBTA42, T30 SMBTA42, T31 SMBTA42, T32 SMBTA42, T33 SMBTA42, T34 SMBTA42, T35 SMBTA42, T36 SMBTA42, T37 SMBTA42, T38 SMBTA42, T39 SMBTA42, T40 SMBTA42, T41 SMBTA42, T42 SMBTA42, T43 SMBTA42, T44 SMBTA42, T45 SMBTA42, T46 SMBTA42, T47 SMBTA42, T48 SMBTA42, T49 SMBTA42

Commit message: Fixed naming
Connections:
- net 4C0 renamed N4_0
- net 4C1 renamed N4_1
- net 4C2 renamed N4_2
- net 4C3 renamed N4_3
- net 4C4 renamed N4_4
- net 4C5 renamed N4_5
- net 4C6 renamed N4_6
- net 4C7 renamed N4_7
- net 4C8 renamed N4_8
- net 4C9 renamed N4_9
Other:
- moved on the sheet: GL1, GL2, N1, N2, N3, N4, R1, R10, R11, R2, R20, R21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
