File: layout/control/c100_rev_b.brd (EAGLE design)
At the start: 100 x 42 mm, 69 parts, among them IC1 STM32F103C8T, IC2 LP2985-SOT23-5, IC3 IC_USBLC6-2, IC4 IC_USBLC6-2, IC5 LT1619ES8, IC6 LP2985-SOT23-5, IC7 IRF7470, T1 LPISR, Y1 532-CRYSTAL, Y2 EQ161-CRYSTAL

Commit message: C100 production ready
Parts:
- removed U$1: (no value), pcb-artwork:JANIS_10MM
- added LOGO2: OSHW_LOGO_FILLX0200-NT, ohw-logo:OSHW_FILLX200_NOTEXT
- moved LOGO1 0.79 mm to (8.00, 1.50)
- moved R20 0.79 mm to (37.8, 15.2)
- moved U$5 0.79 mm to (14.5, 3.25)
Routing:
- net N$17: track 34.1 -> 32.1 mm
Changed lines of the file:
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@@
 <attribute name="VALUE" x="93.385" y="30.655" size="1.27" layer="27" rot="R180"/>
 </element>
-<element name="LOGO1" library="ohw-logo" package="OSHW_FILLX200_NOTEXT" value="OSHW_LOGO_FILLX0200-NT" x="7.25" y="1.25"/>
-<element name="U$5" library="pcb-artwork" package="GITHUB/JAN1S" value="" x="13.75" y="3"/>
+<element name="LOGO1" library="ohw-logo" package="OSHW_FILLX200_NOTEXT" value="OSHW_LOGO_FILLX0200-NT" x="8" y="1.5"/>
+<element name="U$5" library="pcb-artwork" package="GITHUB/JAN1S" value="" x="14.5" y="3.25"/>
 <element name="X1" library="con-cypressindustries" package="32005-201" value="" x="82" y="4.75" smashed="yes" rot="R90">
 <attribute name="OC_NEWARK" value="unknown" x="82" y="4.75" size="1.778" layer="27" rot="R90" display="off"/>
@@
 <attribute name="NAME" x="19.75" y="37.5" size="0.8128" layer="25" rot="R90"/>
 </element>
-<element name="R20" library="rcl" package="R0603" value="8k2" x="37" y="15.5" smashed="yes" rot="R180">
-<attribute name="NAME" x="35.5" y="16" size="0.8128" layer="25" rot="R180"/>
+<element name="R20" library="rcl" package="R0603" value="8k2" x="37.75" y="15.25" smashed="yes" rot="R180">
+<attribute name="NAME" x="36.25" y="15.75" size="0.8128" layer="25" rot="R180"/>
 </element>
 <element name="D2" library="diode" package="SOT23" value="BAT54C" x="24.5" y="27" smashed="yes">
@@
 </element>
 <element name="D3" library="diode" package="DO-214AA" value="ES2" x="30" y="11.5" smashed="yes" rot="R180">
-<attribute name="NAME" x="29.25" y="13.75" size="0.8128" layer="25"/>
+<attribute name="NAME" x="29.25" y="13.5" size="0.8128" layer="25"/>
 </element>
 <element name="C4" library="rcl" package="C2220K" value="1µF/250V" x="36.5" y="9" smashed="yes" rot="R270">
@@
 </element>
 <element name="C17" library="rcl" package="C1210" value="100µF/6.3V" x="30" y="7" smashed="yes">
-<attribute name="NAME" x="31" y="5.25" size="0.8128" layer="25" rot="R180"/>
+<attribute name="NAME" x="29" y="8.5" size="0.8128" layer="25"/>
 </element>
 <element name="R19" library="rcl" package="M1206" value="1M" x="40.5" y="13" smashed="yes" rot="R270">
@@
 <attribute name="NAME" x="87.135" y="19.385" size="0.8128" layer="25" rot="R270"/>
 </element>
-<element name="U$1" library="pcb-artwork" package="JANIS_10MM" value="" x="61" y="5" rot="R45"/>
 <element name="R6" library="rcl" package="R0603" value="1k5" x="85.75" y="11.75" smashed="yes" rot="R270">
 <attribute name="NAME" x="89.615" y="9.615" size="0.8128" layer="25" rot="R90"/>
 </element>
 <element name="BT" library="bt" package="HM-11" value="HM-11" x="40" y="31" smashed="yes">
-<attribute name="NAME" x="35" y="20" size="0.8128" layer="25"/>
-<attribute name="VALUE" x="35" y="21.25" size="0.8128" layer="27"/>
+<attribute name="NAME" x="33.25" y="18.25" size="0.8128" layer="25"/>
+<attribute name="VALUE" x="35" y="20" size="0.8128" layer="27"/>
 </element>
 <element name="C22" library="rcl" package="C0603" value="1µF" x="49" y="21.5" smashed="yes" rot="R90">
@@
 <attribute name="NAME" x="49.885" y="31.135" size="0.8128" layer="25" rot="R270"/>
 </element>
+<element name="LOGO2" library="ohw-logo" package="OSHW_FILLX200_NOTEXT" value="OSHW_LOGO_FILLX0200-NT" x="61.5" y="3" rot="MR0"/>
 </elements>
 <signals>
@@
 <vertex x="47" y="14"/>
 <vertex x="46.5" y="14.5"/>
-<vertex x="29" y="14.5"/>
-<vertex x="27" y="16.5"/>
+<vertex x="29.25" y="14.5"/>
+<vertex x="27.25" y="16.5"/>
 <vertex x="22" y="16.5"/>
 <vertex x="21" y="15.5"/>
@@
 <via x="40" y="6" extent="1-16" drill="0.32"/>
 <via x="16" y="16" extent="1-16" drill="0.32"/>
-<via x="28.5" y="17.5" extent="1-16" drill="0.32"/>
+<via x="29.5" y="15" extent="1-16" drill="0.32"/>
 <via x="20" y="16" extent="1-16" drill="0.32"/>
-<via x="35" y="15" extent="1-16" drill="0.32"/>
-<via x="34" y="16" extent="1-16" drill="0.32"/>
-<via x="30" y="16" extent="1-16" drill="0.32"/>
-<via x="35" y="16" extent="1-16" drill="0.32"/>
+<via x="35.75" y="15" extent="1-16" drill="0.32"/>
+<via x="31" y="15" extent="1-16" drill="0.32"/>
+<via x="35.75" y="15.5" extent="1-16" drill="0.32"/>
 <contactref element="T1" pad="P$2"/>
 <contactref element="TP4" pad="P$1"/>
@@
 <via x="22.5" y="17.5" extent="1-16" drill="0.32"/>
 <via x="15.5" y="24" extent="1-16" drill="0.32"/>
-<via x="25.5" y="17.5" extent="1-16" drill="0.32"/>
+<via x="25" y="17.5" extent="1-16" drill="0.32"/>
 <via x="8" y="20" extent="1-16" drill="0.32"/>
 <contactref element="ISP" pad="2"/>
@@
 <via x="76" y="33.75" extent="1-16" drill="0.32"/>
 <via x="76" y="35.25" extent="1-16" drill="0.32"/>
+<via x="27" y="17.5" extent="1-16" drill="0.32"/>
+<via x="28.25" y="16.25" extent="1-16" drill="0.32"/>
+<via x="26.5" y="21" extent="1-16" drill="0.32"/>
+<via x="26.5" y="25" extent="1-16" drill="0.32"/>
 </signal>
 <signal name="+5V">
@@
 <contactref element="R20" pad="1"/>
 <contactref element="R19" pad="1"/>
-<wire x1="40.5" y1="14.4" x2="40.5" y2="15.5" width="0.254" layer="1"/>
-<wire x1="37.85" y1="15.5" x2="40.5" y2="15.5" width="0.254" layer="1"/>
-<via x="40.5" y="15.5" extent="1-16" drill="0.32"/>
-<wire x1="40.5" y1="15.5" x2="38" y2="15.5" width="0.254" layer="16"/>
-<wire x1="23" y1="28" x2="20.5" y2="30.5" width="0.254" layer="16"/>
+<wire x1="25" y1="26" x2="20.5" y2="30.5" width="0.254" layer="16"/>
 <via x="20.5" y="30.5" extent="1-16" drill="0.32"/>
 <wire x1="20.635" y1="32.1" x2="20.635" y2="30.635" width="0.254" layer="1"/>
 <wire x1="20.635" y1="30.635" x2="20.5" y2="30.5" width="0.254" layer="1"/>
-<wire x1="23" y1="28" x2="25.35" y2="28" width="0.254" layer="16"/>
-<wire x1="25.35" y1="28" x2="37.85" y2="15.5" width="0.254" layer="16"/>
-<wire x1="37.85" y1="15.5" x2="40.5" y2="15.5" width="0.254" layer="16"/>
+<wire x1="38.6" y1="15.9" x2="38.25" y2="16.25" width="0.254" layer="1"/>
+<wire x1="38.25" y1="16.25" x2="30.75" y2="16.25" width="0.254" layer="1"/>
+<wire x1="30.75" y1="16.25" x2="27.5" y2="19.5" width="0.254" layer="1"/>
+<wire x1="27.5" y1="19.5" x2="27.5" y2="25.25" width="0.254" layer="1"/>
+<wire x1="27.5" y1="25.25" x2="26.75" y2="26" width="0.254" layer="1"/>
+<via x="26.75" y="26" extent="1-16" drill="0.32"/>
+<wire x1="26.75" y1="26" x2="25" y2="26" width="0.254" layer="16"/>
+<wire x1="40.5" y1="14.4" x2="40" y2="14.4" width="0.254" layer="1"/>
+<wire x1="38.6" y1="15.9" x2="38.6" y2="15.4" width="0.254" layer="1"/>
+<wire x1="38.6" y1="15.4" x2="38.75" y2="15.25" width="0.254" layer="1"/>
+<wire x1="38.6" y1="15.25" x2="39.15" y2="15.25" width="0.254" layer="1"/>
+<wire x1="39.15" y1="15.25" x2="40" y2="14.4" width="0.254" layer="1"/>
+<wire x1="38.6" y1="15.4" x2="38.6" y2="15.25" width="0" layer="19" extent="1-1"/>
 </signal>
 <signal name="N$19">
