File: layout/control/c100_rev_b.sch (EAGLE design)
At the start: 64 parts, among them IC1 STM32F103C8T, IC2 LP2985-SOT23-5, IC3 IC_USBLC6-2, IC4 IC_USBLC6-2, IC5 LT1619ES8, IC6 LP2985-SOT23-5, IC7 IRF7470, T1 LPISR, X1 MINI-USB-SCHIELD-32005-201, Y1 532-CRYSTAL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

Commit message: Changed structure, added c150 and c200
Parts:
- C18: value 100nF -> 1µF
- C22: value 10µF -> 1µF
Changed lines of the file:
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@@
 <part name="GND15" library="supply1" deviceset="GND" device=""/>
 <part name="GND16" library="supply1" deviceset="GND" device=""/>
-<part name="C18" library="rcl" deviceset="C-EU" device="C0603" value="100nF"/>
+<part name="C18" library="rcl" deviceset="C-EU" device="C0603" value="1µF"/>
 <part name="JP1" library="con-pinhead" deviceset="PINHD-2X5" device="_2.54-SMD"/>
 <part name="GND20" library="supply1" deviceset="GND" device=""/>
@@
 <part name="BT" library="bt" deviceset="HM-11" device=""/>
 <part name="GND32" library="supply1" deviceset="GND" device=""/>
-<part name="C22" library="rcl" deviceset="C-EU" device="C0603" value="10µF"/>
+<part name="C22" library="rcl" deviceset="C-EU" device="C0603" value="1µF"/>
 <part name="+3V4" library="supply1" deviceset="+3V3" device=""/>
 <part name="LED3" library="led" deviceset="LED" device="CHIP-LED0603"/>
