File: layout/control/c150_rev_a.sch (EAGLE design)
At the start: 65 parts, among them IC1 STM32F103C8T, IC2 LP2985-SOT23-5, IC3 IC_USBLC6-2, IC4 IC_USBLC6-2, IC5 LT1619ES8, IC6 LP2985-SOT23-5, IC7 IRF7470, T1 LPISR, X1 MINI-USB-SCHIELD-32005-201, Y1 532-CRYSTAL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

Commit message: C100 production ready
Parts:
- BAT1: value CR1220-HOLDER -> CR2032-HOLDER; device battery-holder:CR1220-HOLDER -> battery-holder:CR2032-HOLDER
Changed lines of the file:
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@@
 <part name="GND13" library="supply1" deviceset="GND" device=""/>
 <part name="GND22" library="supply1" deviceset="GND" device=""/>
-<part name="BAT1" library="battery-holder" deviceset="CR1220-HOLDER" device="" value=""/>
 <part name="R12" library="rcl" deviceset="R-EU_" device="R0603" value="1k"/>
 <part name="R13" library="rcl" deviceset="R-EU_" device="R0603" value="1k"/>
@@
 <part name="GND37" library="supply1" deviceset="GND" device=""/>
 <part name="P+6" library="supply1" deviceset="+5V" device=""/>
+<part name="BAT1" library="battery-holder" deviceset="CR2032-HOLDER" device=""/>
 </parts>
 <sheets>
@@
 <instance part="GND1" gate="1" x="193.04" y="43.18"/>
 <instance part="GND22" gate="1" x="86.36" y="116.84" rot="MR270"/>
-<instance part="BAT1" gate="G$1" x="193.04" y="55.88"/>
 <instance part="+3V8" gate="G$1" x="157.48" y="93.98" rot="R90"/>
 <instance part="IC2" gate="G$1" x="48.26" y="35.56"/>
@@
 <instance part="GND37" gate="1" x="132.08" y="73.66"/>
 <instance part="P+6" gate="1" x="134.62" y="172.72"/>
+<instance part="BAT1" gate="G$1" x="193.04" y="55.88"/>
 </instances>
 <busses>
@@
 <segment>
 <pinref part="GND1" gate="1" pin="GND"/>
-<pinref part="BAT1" gate="G$1" pin="NEG"/>
 <wire x1="193.04" y1="50.8" x2="193.04" y2="48.26" width="0.1524" layer="91"/>
 <pinref part="C11" gate="G$1" pin="2"/>
@@
 <wire x1="210.82" y1="48.26" x2="210.82" y2="53.34" width="0.1524" layer="91"/>
 <junction x="193.04" y="48.26"/>
+<pinref part="BAT1" gate="G$1" pin="NEG"/>
 </segment>
 <segment>
@@
 </segment>
 <segment>
-<pinref part="BAT1" gate="G$1" pin="POS"/>
 <wire x1="193.04" y1="63.5" x2="193.04" y2="66.04" width="0.1524" layer="91"/>
 <pinref part="C11" gate="G$1" pin="1"/>
@@
 <junction x="193.04" y="66.04"/>
 <label x="193.04" y="68.58" size="1.778" layer="95"/>
-</segment>
-</net>
+<pinref part="BAT1" gate="G$1" pin="POS"/>
+</segment>
+</net>
