File: layout/control/c150_rev_a.brd (EAGLE design)
At the start: 150 x 42 mm, 71 parts, among them IC1 STM32F103C8T, IC2 LP2985-SOT23-5, IC3 IC_USBLC6-2, IC4 IC_USBLC6-2, IC5 LT1619ES8, IC6 LP2985-SOT23-5, IC7 IRF7470, T1 LPISR, Y1 532-CRYSTAL, Y2 EQ161-CRYSTAL

Commit message: C100 production ready
Parts:
- BAT1: value (none) -> CR2032-HOLDER; device battery-holder:HARWIN-CR1220 -> battery-holder:CH28-2032LF
- moved BT 32.0 mm to (58.0, 31.0)
- moved C22 32.0 mm to (67.0, 21.5)
- moved LED3 32.0 mm to (68.5, 27.2)
- moved R7 32.0 mm to (67.0, 27.2)
- moved R8 32.0 mm to (67.0, 30.5)
- moved BAT1 17.0 mm to (96.0, 28.0), turned to 270 degrees
- moved U$1 0.50 mm to (69.5, 7.00)
Routing:
- net USART2_RX: track 47.7 -> 88.6 mm, vias 2 -> 0
- net USART2_TX: track 48.3 -> 88.5 mm
- net BT_USER: track 38.1 -> 78.3 mm
- net +3V3: track 103.3 -> 137.7 mm
- net VBAT: track 21.1 -> 32.0 mm

Commit message: Finished c150 rev a
Parts:
- moved R20 0.79 mm to (37.8, 15.2)
Routing:
- net N$17: track 34.1 -> 33.4 mm
- net HV_EN: track 126.3 -> 126.8 mm
Changed lines of the file:
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@@
 <attribute name="NAME" x="19.75" y="37.5" size="0.8128" layer="25" rot="R90"/>
 </element>
-<element name="R20" library="rcl" package="R0603" value="8k2" x="37" y="15.5" smashed="yes" rot="R180">
-<attribute name="NAME" x="35.5" y="16" size="0.8128" layer="25" rot="R180"/>
+<element name="R20" library="rcl" package="R0603" value="8k2" x="37.75" y="15.25" smashed="yes" rot="R180">
+<attribute name="NAME" x="36.25" y="15.75" size="0.8128" layer="25" rot="R180"/>
 </element>
 <element name="D2" library="diode" package="SOT23" value="BAT54C" x="24.5" y="27" smashed="yes">
@@
 <polygon width="0.254" layer="1" rank="5">
 <vertex x="3" y="42"/>
-<vertex x="30" y="42"/>
-<vertex x="32" y="40"/>
-<vertex x="32" y="33"/>
-<vertex x="33" y="32"/>
+<vertex x="24" y="42"/>
+<vertex x="26" y="40"/>
+<vertex x="26" y="33"/>
+<vertex x="27" y="32"/>
 <vertex x="83" y="32"/>
 <vertex x="84" y="33"/>
@@
 <polygon width="0.254" layer="16">
 <vertex x="3" y="42"/>
-<vertex x="30" y="42"/>
-<vertex x="32" y="40"/>
-<vertex x="32" y="33"/>
-<vertex x="33" y="32"/>
+<vertex x="24" y="42"/>
+<vertex x="26" y="40"/>
+<vertex x="26" y="33"/>
+<vertex x="27" y="32"/>
 <vertex x="83" y="32"/>
 <vertex x="84" y="33"/>
@@
 <via x="40" y="6" extent="1-16" drill="0.32"/>
 <via x="16" y="16" extent="1-16" drill="0.32"/>
-<via x="28.5" y="17.5" extent="1-16" drill="0.32"/>
+<via x="27" y="17.5" extent="1-16" drill="0.32"/>
 <via x="20" y="16" extent="1-16" drill="0.32"/>
-<via x="35" y="15" extent="1-16" drill="0.32"/>
-<via x="34" y="16" extent="1-16" drill="0.32"/>
-<via x="30" y="16" extent="1-16" drill="0.32"/>
-<via x="35" y="16" extent="1-16" drill="0.32"/>
+<via x="35.75" y="15" extent="1-16" drill="0.32"/>
+<via x="31" y="15" extent="1-16" drill="0.32"/>
+<via x="35.75" y="15.5" extent="1-16" drill="0.32"/>
 <contactref element="T1" pad="P$2"/>
 <contactref element="TP4" pad="P$1"/>
@@
 <via x="22.5" y="17.5" extent="1-16" drill="0.32"/>
 <via x="15.5" y="24" extent="1-16" drill="0.32"/>
-<via x="25.5" y="17.5" extent="1-16" drill="0.32"/>
+<via x="24.75" y="17.5" extent="1-16" drill="0.32"/>
 <via x="8" y="20" extent="1-16" drill="0.32"/>
 <contactref element="ISP" pad="2"/>
@@
 <via x="56" y="20" extent="1-16" drill="0.32"/>
 <via x="60" y="24" extent="1-16" drill="0.32"/>
-<via x="31" y="39" extent="1-16" drill="0.32"/>
-<via x="31" y="37" extent="1-16" drill="0.32"/>
-<via x="32" y="32" extent="1-16" drill="0.32"/>
-<via x="33" y="31" extent="1-16" drill="0.32"/>
-<via x="31" y="35" extent="1-16" drill="0.32"/>
-<via x="31" y="33" extent="1-16" drill="0.32"/>
-<via x="35" y="31" extent="1-16" drill="0.32"/>
+<via x="25" y="39" extent="1-16" drill="0.32"/>
+<via x="25" y="37" extent="1-16" drill="0.32"/>
+<via x="26" y="32" extent="1-16" drill="0.32"/>
+<via x="27" y="31" extent="1-16" drill="0.32"/>
+<via x="25" y="35" extent="1-16" drill="0.32"/>
+<via x="25" y="33" extent="1-16" drill="0.32"/>
+<via x="29" y="31" extent="1-16" drill="0.32"/>
 <via x="37" y="31" extent="1-16" drill="0.32"/>
 <via x="39" y="31" extent="1-16" drill="0.32"/>
@@
 <via x="126" y="35.25" extent="1-16" drill="0.32"/>
 <via x="24" y="40" extent="1-16" drill="0.32"/>
-<via x="26" y="40" extent="1-16" drill="0.32"/>
-<via x="28" y="40" extent="1-16" drill="0.32"/>
-<via x="30" y="40" extent="1-16" drill="0.32"/>
+<via x="33" y="31" extent="1-16" drill="0.32"/>
+<via x="31" y="31" extent="1-16" drill="0.32"/>
+<via x="35" y="31" extent="1-16" drill="0.32"/>
 <contactref element="JP1" pad="4"/>
 <contactref element="JP1" pad="6"/>
@@
 <via x="64" y="16" extent="1-16" drill="0.32"/>
 <via x="24" y="20" extent="1-16" drill="0.32"/>
-<via x="28" y="20" extent="1-16" drill="0.32"/>
-<via x="28" y="24" extent="1-16" drill="0.32"/>
+<via x="27.5" y="20" extent="1-16" drill="0.32"/>
+<via x="27.5" y="24" extent="1-16" drill="0.32"/>
 <via x="56" y="12" extent="1-16" drill="0.32"/>
 <via x="60" y="12" extent="1-16" drill="0.32"/>
@@
 <via x="66.5" y="25.25" extent="1-16" drill="0.32"/>
 <via x="66.5" y="24.75" extent="1-16" drill="0.32"/>
+<via x="29.5" y="15" extent="1-16" drill="0.32"/>
+<via x="28.25" y="16.25" extent="1-16" drill="0.32"/>
 </signal>
 <signal name="+5V">
@@
 <wire x1="31.25" y1="17.75" x2="49.25" y2="17.75" width="0.254" layer="1"/>
 <wire x1="49.25" y1="17.75" x2="53" y2="14" width="0.254" layer="1"/>
-<via x="53" y="14" extent="1-16" drill="0.32"/>
-<wire x1="53" y1="14" x2="105" y2="14" width="0.254" layer="16"/>
-<wire x1="105" y1="14" x2="106.75" y2="12.25" width="0.254" layer="16"/>
+<wire x1="104" y1="14.75" x2="106.75" y2="12.25" width="0.254" layer="16"/>
 <wire x1="106.75" y1="13" x2="106.75" y2="12.25" width="0.254" layer="1"/>
 <via x="106.75" y="12.25" extent="1-16" drill="0.32"/>
+<wire x1="53" y1="14" x2="103.25" y2="14" width="0.254" layer="1"/>
+<wire x1="103.25" y1="14" x2="104" y2="14.75" width="0.254" layer="1"/>
+<via x="104" y="14.75" extent="1-16" drill="0.32"/>
 </signal>
 <signal name="RESET">
@@
 <contactref element="R20" pad="1"/>
 <contactref element="R19" pad="1"/>
-<wire x1="40.5" y1="14.4" x2="40.5" y2="15.5" width="0.254" layer="1"/>
-<wire x1="37.85" y1="15.5" x2="40.5" y2="15.5" width="0.254" layer="1"/>
-<via x="40.5" y="15.5" extent="1-16" drill="0.32"/>
-<wire x1="40.5" y1="15.5" x2="38" y2="15.5" width="0.254" layer="16"/>
-<wire x1="23" y1="28" x2="20.5" y2="30.5" width="0.254" layer="16"/>
+<wire x1="25" y1="26" x2="20.5" y2="30.5" width="0.254" layer="16"/>
 <via x="20.5" y="30.5" extent="1-16" drill="0.32"/>
 <wire x1="20.635" y1="32.1" x2="20.635" y2="30.635" width="0.254" layer="1"/>
 <wire x1="20.635" y1="30.635" x2="20.5" y2="30.5" width="0.254" layer="1"/>
-<wire x1="23" y1="28" x2="25.35" y2="28" width="0.254" layer="16"/>
-<wire x1="25.35" y1="28" x2="37.85" y2="15.5" width="0.254" layer="16"/>
-<wire x1="37.85" y1="15.5" x2="40.5" y2="15.5" width="0.254" layer="16"/>
+<wire x1="38.6" y1="15.25" x2="38.6" y2="15.9" width="0.254" layer="1"/>
+<wire x1="38.6" y1="15.9" x2="38.25" y2="16.25" width="0.254" layer="1"/>
+<wire x1="38.25" y1="16.25" x2="30.5" y2="16.25" width="0.254" layer="1"/>
+<wire x1="30.5" y1="16.25" x2="28.5" y2="18.25" width="0.254" layer="1"/>
+<wire x1="28.5" y1="18.25" x2="28.5" y2="25.5" width="0.254" layer="1"/>
+<wire x1="28.5" y1="25.5" x2="27.75" y2="26.25" width="0.254" layer="1"/>
+<wire x1="27.75" y1="26.25" x2="27.25" y2="26.25" width="0.254" layer="1"/>
+<wire x1="27.25" y1="26.25" x2="27" y2="26" width="0.254" layer="1"/>
+<via x="27" y="26" extent="1-16" drill="0.32"/>
+<wire x1="27" y1="26" x2="25" y2="26" width="0.254" layer="16"/>
+<wire x1="38.6" y1="15.25" x2="38.6" y2="15.15" width="0.254" layer="1"/>
+<wire x1="38.6" y1="15.15" x2="38.75" y2="15" width="0.254" layer="1"/>
+<wire x1="38.75" y1="15" x2="40.25" y2="15" width="0.254" layer="1"/>
+<wire x1="40.25" y1="15" x2="40.5" y2="14.75" width="0.254" layer="1"/>
+<wire x1="40.5" y1="14.4" x2="40.5" y2="14.75" width="0.254" layer="1"/>
 </signal>
 <signal name="N$19">
@@
 <wire x1="135.25" y1="31.25" x2="130.75" y2="31.25" width="0.3048" layer="16"/>
 <wire x1="130.75" y1="31.25" x2="129.25" y2="32.75" width="0.3048" layer="16"/>
-<wire x1="129.25" y1="32.75" x2="121" y2="32.75" width="0.3048" layer="16"/>
-<via x="121" y="32.75" extent="1-16" drill="0.32"/>
+<wire x1="129.25" y1="32.75" x2="122" y2="32.75" width="0.3048" layer="16"/>
+<via x="122" y="32.75" extent="1-16" drill="0.32"/>
 <contactref element="BAT1" pad="POS"/>
-<wire x1="121" y1="32.75" x2="111.75" y2="32.75" width="0.3048" layer="1"/>
+<wire x1="122" y1="32.75" x2="111.75" y2="32.75" width="0.3048" layer="1"/>
 <wire x1="111.75" y1="32.75" x2="110.65" y2="31.65" width="0.3048" layer="1"/>
 <wire x1="110.65" y1="28" x2="110.65" y2="31.65" width="0.3048" layer="1"/>
