File: layout/control/c200_rev_a.brd (EAGLE design)
At the start: 200 x 50 mm, 77 parts, among them IC1 STM32F103C8T, IC2 LP2985-SOT23-5, IC3 IC_USBLC6-2, IC4 IC_USBLC6-2, IC5 LT1619ES8, IC6 LP2985-SOT23-5, IC7 IRF7470, T1 LPISR, Y1 532-CRYSTAL, Y2 EQ161-CRYSTAL

Commit message: Added final c200 production files
Parts:
- moved R9 24.4 mm to (127.0, 24.5), turned to 0 degrees
- moved LOGO2 11.0 mm to (75.2, 3.25)
- moved U$5 11.0 mm to (81.8, 5.00)
- moved U$1 10.8 mm to (83.0, 7.00)
- moved C18 1.00 mm to (175.5, 30.8)
- moved BAT1 0.71 mm to (163.5, 27.5)
- renumbered U$3 to WIFI
Routing:
- net RFMOD_RST: track 4.27 -> 111.1 mm, vias 0 -> 4
- net RFMOD_FLASH: track 3.65 -> 74.2 mm, vias 0 -> 4
- net RFMOD_DBG: track 3.65 -> 73.6 mm, vias 0 -> 4
- net +3V3: track 103.3 -> 157.0 mm
- net RFMOD_EN: track 38.1 -> 83.7 mm
- net VBAT: track 21.1 -> 20.6 mm
