File: layout/control/c200_rev_a.sch (EAGLE design)
At the start: 71 parts, among them IC1 STM32F103C8T, IC2 LP2985-SOT23-5, IC3 IC_USBLC6-2, IC4 IC_USBLC6-2, IC5 LT1619ES8, IC6 LP2985-SOT23-5, IC7 IRF7470, T1 LPISR, X1 MINI-USB-SCHIELD-32005-201, Y1 532-CRYSTAL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

Commit message: Added final c200 production files
Parts:
- renumbered U$3 to WIFI
Changed lines of the file:
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@@
 <?xml version="1.0" encoding="utf-8"?>
 <!DOCTYPE eagle SYSTEM "eagle.dtd">
-<eagle version="7.6.0">
+<eagle version="6.1">
 <drawing>
 <settings>
@@
 <part name="GND37" library="supply1" deviceset="GND" device=""/>
 <part name="P+6" library="supply1" deviceset="+5V" device=""/>
-<part name="U$3" library="espressif" deviceset="ESP-12F" device=""/>
+<part name="WIFI" library="espressif" deviceset="ESP-12F" device=""/>
 <part name="C23" library="rcl" deviceset="C-EU" device="C0603" value="1µF"/>
 <part name="GND17" library="supply1" deviceset="GND" device=""/>
@@
 <instance part="GND37" gate="1" x="132.08" y="73.66"/>
 <instance part="P+6" gate="1" x="134.62" y="172.72"/>
-<instance part="U$3" gate="G$1" x="421.64" y="76.2"/>
+<instance part="WIFI" gate="G$1" x="421.64" y="76.2"/>
 <instance part="C23" gate="G$1" x="449.58" y="58.42"/>
 <instance part="GND17" gate="1" x="449.58" y="48.26"/>
@@
 </segment>
 <segment>
-<pinref part="U$3" gate="G$1" pin="GND"/>
+<pinref part="WIFI" gate="G$1" pin="GND"/>
 <pinref part="C23" gate="G$1" pin="2"/>
 <wire x1="439.42" y1="53.34" x2="449.58" y2="53.34" width="0.1524" layer="91"/>
@@
 </segment>
 <segment>
-<pinref part="U$3" gate="G$1" pin="VCC"/>
+<pinref part="WIFI" gate="G$1" pin="VCC"/>
 <pinref part="C23" gate="G$1" pin="1"/>
 <wire x1="439.42" y1="60.96" x2="449.58" y2="60.96" width="0.1524" layer="91"/>
@@
 </segment>
 <segment>
-<pinref part="U$3" gate="G$1" pin="RXD"/>
+<pinref part="WIFI" gate="G$1" pin="RXD"/>
 <wire x1="439.42" y1="71.12" x2="441.96" y2="71.12" width="0.1524" layer="91"/>
 <label x="441.96" y="71.12" size="1.778" layer="95"/>
@@
 </segment>
 <segment>
-<pinref part="U$3" gate="G$1" pin="TXD"/>
+<pinref part="WIFI" gate="G$1" pin="TXD"/>
 <wire x1="439.42" y1="73.66" x2="441.96" y2="73.66" width="0.1524" layer="91"/>
 <label x="441.96" y="73.66" size="1.778" layer="95"/>
@@
 </segment>
 <segment>
-<pinref part="U$3" gate="G$1" pin="GPIO2"/>
+<pinref part="WIFI" gate="G$1" pin="GPIO2"/>
 <pinref part="R11" gate="G$1" pin="1"/>
 <wire x1="403.86" y1="68.58" x2="393.7" y2="68.58" width="0.1524" layer="91"/>
@@
 </segment>
 <segment>
-<pinref part="U$3" gate="G$1" pin="EN"/>
+<pinref part="WIFI" gate="G$1" pin="EN"/>
 <wire x1="439.42" y1="91.44" x2="462.28" y2="91.44" width="0.1524" layer="91"/>
 <label x="462.28" y="91.44" size="1.778" layer="95"/>
@@
 <net name="RFMOD_RST" class="0">
 <segment>
-<pinref part="U$3" gate="G$1" pin="RST"/>
+<pinref part="WIFI" gate="G$1" pin="RST"/>
 <wire x1="439.42" y1="96.52" x2="452.12" y2="96.52" width="0.1524" layer="91"/>
 <label x="462.28" y="96.52" size="1.778" layer="95"/>
@@
 <net name="RFMOD_FLASH" class="0">
 <segment>
-<pinref part="U$3" gate="G$1" pin="GPIO0"/>
+<pinref part="WIFI" gate="G$1" pin="GPIO0"/>
 <pinref part="R10" gate="G$1" pin="1"/>
 <wire x1="403.86" y1="66.04" x2="383.54" y2="66.04" width="0.1524" layer="91"/>
@@
 <net name="N$6" class="0">
 <segment>
-<pinref part="U$3" gate="G$1" pin="GPIO15"/>
+<pinref part="WIFI" gate="G$1" pin="GPIO15"/>
 <pinref part="R14" gate="G$1" pin="1"/>
 <wire x1="398.78" y1="93.98" x2="403.86" y2="93.98" width="0.1524" layer="91"/>
